Commit message: Fix wheel positioning, decimate ugv mesh, use package:// paths
- Fix wheel rotation offset (xyz now compensates for R_z rotation per side)
- Move wheels 30mm outward (10mm half-profile + 20mm suspension gap)
- Decimate ugv.stl from 42MB to 2.1MB (862K→43K faces)
- Switch mesh_dir from absolute file:// to package:// for Jetson portability
- Add RViz config with pre-set Fixed Frame and RobotModel settings
- Add __pycache__ to .gitignore

Co-Authored-By: Claude Opus 4.6 (1M context) <noreply@anthropic.com>

File: struktura/urdf/qubertmk1.urdf.xacro (robot description, xacro)
@@ -29,5 +29,5 @@
   <!-- Wheel positions (from chassis center, at bottom frame corners) -->
   <xacro:property name="wheel_x" value="${crossbar_offset}"/>
-  <xacro:property name="wheel_y" value="${cube_outer / 2 + 0.05}"/>  <!-- offset outward from frame -->
+  <xacro:property name="wheel_y" value="${cube_outer / 2 + 0.030}"/>  <!-- frame edge + 10mm half-profile + 20mm suspension gap -->
   <xacro:property name="wheel_z" value="${-cube_outer / 2}"/>
   <!-- RoArm-M2-S dimensions (approximate) -->
@@ -78,5 +78,5 @@
   </xacro:macro>
   <!-- Mesh base path -->
-  <xacro:property name="mesh_dir" value="file:///home/marko/Documents/00 mirko 3d print/000qubertmk1-20260324T182111Z-1-001/000qubertmk1/struktura/meshes"/>
+  <xacro:property name="mesh_dir" value="package://qubertmk1_description/meshes"/>
   <!-- Profile bar macro: mesh is along Z in STL, centered at (128,128,L/2) mm -->
   <!-- We rotate Z→X (rpy 0 pi/2 0) and shift to center at link origin -->
@@ -127,10 +127,12 @@
   <!-- Wheel + suspension macro (ugv.stl includes wheel + suspension as one piece) -->
   <!-- ugv.stl bounds: (88.3,77.7,0)→(167.7,178.3,100.7) mm, center ~(128,128,50) mm -->
-  <!-- Right side (y_sign=-1): rotate pi around Z (clockwise when viewed from top) -->
-  <!-- Left side  (y_sign=+1): no rotation (anticlockwise / mirrored) -->
+  <!-- URDF visual: first rotates mesh by rpy, THEN translates by xyz -->
+  <!-- So xyz must be: -R_z(angle) * mesh_center to re-center after rotation -->
+  <!-- Left (y_sign=+1): R_z(+pi/2) → center goes to (-0.128, 0.128) → xyz=(0.128, -0.128) -->
+  <!-- Right(y_sign=-1): R_z(-pi/2) → center goes to (0.128, -0.128) → xyz=(-0.128, 0.128) -->
   <xacro:macro name="wheel_assembly" params="prefix x_sign y_sign">
     <link name="${prefix}_suspension">
       <visual>
-        <origin xyz="-0.128 -0.128 -0.050" rpy="0 0 ${y_sign * pi/2 - pi/2}"/>
+        <origin xyz="${y_sign * 0.128} ${-y_sign * 0.128} -0.050" rpy="0 0 ${y_sign * pi/2}"/>
         <geometry>
           <mesh filename="${mesh_dir}/chassis/ugv.stl" scale="0.001 0.001 0.001"/>
